File: IGN6.kicad_sch (KiCad schematic)
At the start: 24 parts

Commit message: Remove dumb-coil IGBTs and route the AMPSEAL header pins.
Drop Q7-Q12 from the ignition sheet and the board, track every J30/J31 signal pad to existing copper, and document the remaining KiCad 8 fab steps.

Co-authored-by: Quintin <quintinbannink42@users.noreply.github.com>
Parts:
- Q? (x6): MyComment DNP -> REMOVED smart-coil-only; now not fitted; now left out of the parts list
Changed lines of the file:
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@@
 		(unit 1)
 		(exclude_from_sim no)
-		(in_bom yes)
-		(on_board yes)
-		(dnp no)
+		(in_bom no)
+		(on_board no)
+		(dnp yes)
 		(property "Reference" "Q?"
 			(at 115.7986 124.5616 0)
@@
 			)
 		)
-		(property "MyComment" "DNP"
+		(property "MyComment" "REMOVED smart-coil-only"
 			(at 114.3 129.54 0)
 			(effects
@@
 		(unit 1)
 		(exclude_from_sim no)
-		(in_bom yes)
-		(on_board yes)
-		(dnp no)
+		(in_bom no)
+		(on_board no)
+		(dnp yes)
 		(property "Reference" "Q?"
 			(at 115.7986 68.6816 0)
@@
 			)
 		)
-		(property "MyComment" "DNP"
+		(property "MyComment" "REMOVED smart-coil-only"
 			(at 114.3 73.66 0)
 			(effects
@@
 		(unit 1)
 		(exclude_from_sim no)
-		(in_bom yes)
-		(on_board yes)
-		(dnp no)
+		(in_bom no)
+		(on_board no)
+		(dnp yes)
 		(property "Reference" "Q?"
 			(at 115.7986 96.6216 0)
@@
 			)
 		)
-		(property "MyComment" "DNP"
+		(property "MyComment" "REMOVED smart-coil-only"
 			(at 114.3 101.6 0)
 			(effects
@@
 		(unit 1)
 		(exclude_from_sim no)
-		(in_bom yes)
-		(on_board yes)
-		(dnp no)
+		(in_bom no)
+		(on_board no)
+		(dnp yes)
 		(property "Reference" "Q?"
 			(at 162.7886 68.6816 0)
@@
 			)
 		)
-		(property "MyComment" "DNP"
+		(property "MyComment" "REMOVED smart-coil-only"
 			(at 161.29 73.66 0)
 			(effects
@@
 		(unit 1)
 		(exclude_from_sim no)
-		(in_bom yes)
-		(on_board yes)
-		(dnp no)
+		(in_bom no)
+		(on_board no)
+		(dnp yes)
 		(property "Reference" "Q?"
 			(at 162.7886 124.5616 0)
@@
 			)
 		)
-		(property "MyComment" "DNP"
+		(property "MyComment" "REMOVED smart-coil-only"
 			(at 161.29 129.54 0)
 			(effects
@@
 		(unit 1)
 		(exclude_from_sim no)
-		(in_bom yes)
-		(on_board yes)
-		(dnp no)
+		(in_bom no)
+		(on_board no)
+		(dnp yes)
 		(property "Reference" "Q?"
 			(at 162.7886 96.6216 0)
@@
 			)
 		)
-		(property "MyComment" "DNP"
+		(property "MyComment" "REMOVED smart-coil-only"
 			(at 161.29 101.6 0)
 			(effects
