File: uaefi.kicad_sch (KiCad schematic)
At the start: 68 parts, among them J1 Conn_02x02_Odd_Even, J1 USB_B_Mini, J1 USB_C, J10 5569-16A2, J11 Conn_02x02_Odd_Even, J12 Conn_02x02_Odd_Even, J13 Conn_02x02_Odd_Even, J14 Conn_02x02_Odd_Even, J15 Conn_02x02_Odd_Even, J16 Conn_02x02_Odd_Even, J17 Conn_01x06, J17 Conn_02x02_Odd_Even, J18 Conn_02x02_Odd_Even, J19 Conn_02x02_Odd_Even, J2 5569-20A2, J20 Conn_02x02_Odd_Even, J21 Conn_02x02_Odd_Even, J22 Conn_02x02_Odd_Even, J24 Conn_02x02_Odd_Even, J3 5569-06A2, J4 5569-08A2, J5 5569-18A2, J5 Conn_01x05_Male, M1 Module-power_12and5V-0.3, M3 Module-knock-0.2, M3 Module-vr-discrete-0.5, M4 Module-vr-max9924-0.1, M5 Module-wbo-0.5, M6 Module:mega-mcu100/0.3, M7 Module-can-0.1, P1 Pad, P2 Pad, P3 Pad, P4 Pad, P5 Pad, P6 Pad, P7 Pad, P8 Pad, U4 JDY-33

Commit message: Replace Mini-Fit harness connectors with two AMPSEAL 35 headers.
Map rev E loom nets onto J30 and J31, document the pinout, and place unverified 776163-1 footprints without re-routing.

Co-authored-by: Quintin <quintinbannink42@users.noreply.github.com>
Parts:
- added J30: AMPSEAL-A 776163-1, ampseal:TE_AMPSEAL_35_776163-1, symbol Connector:AMPSEAL_35_776163-1
- added J31: AMPSEAL-B 776163-1, ampseal:TE_AMPSEAL_35_776163-1, symbol Connector:AMPSEAL_35_776163-1
- J10, J2, J3, J4, J5: now not fitted
Connections:
- net +12V: now also J30.32 (Pin_32)
- net +12V_RAW: now also J30.33 (Pin_33)
- net +5VP: now also J31.31 (Pin_31), J31.32 (Pin_32), J31.33 (Pin_33)
- net 12V_KEY: now also J30.31 (Pin_31)
- net CAN+: now also J31.25 (Pin_25)
- net CAN-: now also J31.24 (Pin_24)
- net EGT+: now also J31.1 (Pin_1)
- net GND: now also J30.28 (Pin_28), J30.29 (Pin_29), J30.30 (Pin_30), J31.26 (Pin_26)
- net GNDA: now also J31.27 (Pin_27), J31.28 (Pin_28), J31.29 (Pin_29), J31.30 (Pin_30)
- net IN_AUX1: now also J31.14 (Pin_14)
- net IN_AUX2: now also J31.13 (Pin_13)
- net IN_AUX3: now also J31.12 (Pin_12)
- net IN_BUTTON1: now also J31.11 (Pin_11)
- net IN_BUTTON2: now also J31.10 (Pin_10)
- net IN_BUTTON3: now also J31.9 (Pin_9)
- net IN_CLT: now also J31.17 (Pin_17)
- net IN_FLEX: now also J31.16 (Pin_16)
- net IN_HALL1: now also J31.8 (Pin_8)
- net IN_HALL2: now also J31.7 (Pin_7)
- net IN_HALL3: now also J31.6 (Pin_6)
- net IN_IAT: now also J31.18 (Pin_18)
- net IN_KNOCK_RAW: now also J31.15 (Pin_15)
- net IN_MAP: now also J31.23 (Pin_23)
- net IN_PPS1: now also J31.20 (Pin_20)
- net IN_PPS2: now also J31.19 (Pin_19)
- net IN_TPS1: now also J31.22 (Pin_22)
- net IN_TPS2: now also J31.21 (Pin_21)
- net OUT_DC1+: now also J30.9 (Pin_9)
- net OUT_DC1-: now also J30.8 (Pin_8)
- net OUT_DC2+: now also J30.7 (Pin_7)
- net OUT_DC2-: now also J30.6 (Pin_6)
- net OUT_IGN1: now also J30.21 (Pin_21)
- net OUT_IGN2: now also J30.20 (Pin_20)
- net OUT_IGN3: now also J30.19 (Pin_19)
- net OUT_IGN4: now also J30.18 (Pin_18)
- net OUT_IGN5: now also J30.17 (Pin_17)
- net OUT_IGN6: now also J30.16 (Pin_16)
- net OUT_INJ1: now also J30.27 (Pin_27)
- net OUT_INJ2: now also J30.26 (Pin_26)
- net OUT_INJ3: now also J30.25 (Pin_25)
- net OUT_INJ4: now also J30.24 (Pin_24)
- net OUT_INJ5: now also J30.23 (Pin_23)
- net OUT_INJ6: now also J30.22 (Pin_22)
- net OUT_LS1: now also J30.15 (Pin_15)
- net OUT_LS2: now also J30.14 (Pin_14)
- net OUT_LS3: now also J30.13 (Pin_13)
- net OUT_LS4: now also J30.12 (Pin_12)
- net OUT_LS_HOT1: now also J30.11 (Pin_11)
- net OUT_LS_HOT2: now also J30.10 (Pin_10)
- net VR_DISCRETE+: now also J31.3 (Pin_3)
- net VR_DISCRETE-: now also J31.2 (Pin_2)
- net VR_MAX9924+: now also J31.5 (Pin_5)
- net VR_MAX9924-: now also J31.4 (Pin_4)
- net WBO_Heater: now also J30.5 (Pin_5)
- net WBO_Ip: now also J30.4 (Pin_4)
- net WBO_Rtrim: now also J30.1 (Pin_1)
- net WBO_Un: now also J30.3 (Pin_3)
- net WBO_Vm: now also J30.2 (Pin_2)
Other:
- note added: "Dual AMPSEAL 35 redesign: J30 connector A (outputs/power/WBO), J31 connector B (sensors/CAN). Molex Mini-Fit J2 J3 J4 J5 J10 are DNP. Pinout: docs/ampseal-35-pinout.md. Footprint pad geometry is a hypothesis."

Commit message: Replace dual AMPSEAL headers with one SUPERSEAL 60.
J30 is a TE 6437288-5 on the grown right edge. The AMPSEAL headers and the 2.54 mm 2x02 sockets are removed. Harness tracks are sized for the 1 oz neck, not the 15 A catalog figure. Twenty-one header pads are still unconnected.

Co-authored-by: Quintin <quintinbannink42@users.noreply.github.com>
Parts:
- removed J1: USB_C, kicad6-libraries:USB_C, symbol misc:USB_C
- removed J1: USB_B_Mini, hellen-one-common:USB-MINI-B-VERTICAL, symbol hellen-one-common:USB_B_Mini
- removed J1, J11, J12, J13, J14, J15, J16, J17, J18, J19, J20, J21, J22, J24: Conn_02x02_Odd_Even, Connector_PinSocket_2.54mm:PinSocket_2x02_P2.54mm_Vertical, symbol Connector_Generic:Conn_02x02_Odd_Even
- removed J17: Conn_01x06, Connector_PinHeader_2.54mm:PinHeader_1x06_P2.54mm_Vertical, symbol Connector_Generic:Conn_01x06
- removed J30: AMPSEAL-A 776163-1, ampseal:TE_AMPSEAL_35_776163-1, symbol Connector:AMPSEAL_35_776163-1
- removed J31: AMPSEAL-B 776163-1, ampseal:TE_AMPSEAL_35_776163-1, symbol Connector:AMPSEAL_35_776163-1
- added J30: 6437288-5, local-conn:TE_6437288-5_SuperSeal_60_RA, symbol Connector:SUPERSEAL_60_6437288-5
Connections:
- net +12V: now also J30.1 (+12V)
- net +12V_RAW: now also J30.2 (+12V_RAW)
- net +5VP: now also J30.7 (+5VP)
- net 12V_KEY: now also J30.3 (12V_KEY)
- net CAN+: now also J30.9 (CAN+)
- net CAN-: now also J30.35 (CAN-)
- net EGT+: now also J30.36 (EGT+)
- net EGT-: now also J30.37 (EGT-)
- net GND: now also J30.4 (GND), J30.5 (GND)
- net GNDA: now also J30.8 (GNDA)
- net IN_AUX1: now also J30.23 (IN_AUX1)
- net IN_AUX2: now also J30.24 (IN_AUX2)
- net IN_AUX3: now also J30.25 (IN_AUX3)
- net IN_BUTTON1: now also J30.42 (IN_BUTTON1)
- net IN_BUTTON2: now also J30.43 (IN_BUTTON2)
- net IN_BUTTON3: now also J30.44 (IN_BUTTON3)
- net IN_CLT: now also J30.20 (IN_CLT)
- net IN_FLEX: now also J30.21 (IN_FLEX)
- net IN_HALL1: now also J30.45 (IN_HALL1)
- net IN_HALL2: now also J30.46 (IN_HALL2)
- net IN_HALL3: now also J30.47 (IN_HALL3)
- net IN_IAT: now also J30.19 (IN_IAT)
- net IN_KNOCK_RAW: now also J30.22 (IN_KNOCK_RAW)
- net IN_MAP: now also J30.14 (IN_MAP)
- net IN_PPS1: now also J30.17 (IN_PPS1)
- net IN_PPS2: now also J30.18 (IN_PPS2)
- net IN_TPS1: now also J30.15 (IN_TPS1)
- net IN_TPS2: now also J30.16 (IN_TPS2)
- net OUT_DC1+: now also J30.32 (OUT_DC1+)
- net OUT_DC1-: now also J30.33 (OUT_DC1-)
- net OUT_DC2+: now also J30.34 (OUT_DC2+)
- net OUT_DC2-: now also J30.54 (OUT_DC2-)
- net OUT_IGN1: now also J30.48 (OUT_IGN1)
- net OUT_IGN2: now also J30.49 (OUT_IGN2)
- net OUT_IGN3: now also J30.50 (OUT_IGN3)
- net OUT_IGN4: now also J30.51 (OUT_IGN4)
- net OUT_IGN5: now also J30.52 (OUT_IGN5)
- net OUT_IGN6: now also J30.53 (OUT_IGN6)
- net OUT_INJ1: now also J30.26 (OUT_INJ1)
- net OUT_INJ2: now also J30.27 (OUT_INJ2)
- net OUT_INJ3: now also J30.28 (OUT_INJ3)
- net OUT_INJ4: now also J30.29 (OUT_INJ4)
- net OUT_INJ5: now also J30.30 (OUT_INJ5)
- net OUT_INJ6: now also J30.31 (OUT_INJ6)
- net OUT_LS1: now also J30.55 (OUT_LS1)
- net OUT_LS2: now also J30.56 (OUT_LS2)
- net OUT_LS3: now also J30.57 (OUT_LS3)
- net OUT_LS4: now also J30.58 (OUT_LS4)
- net OUT_LS_HOT1: now also J30.59 (OUT_LS_HOT1)
- net OUT_LS_HOT2: now also J30.60 (OUT_LS_HOT2)
- net VR_DISCRETE+: now also J30.40 (VR_DISCRETE+)
- net VR_DISCRETE-: now also J30.41 (VR_DISCRETE-)
- net VR_MAX9924+: now also J30.38 (VR_MAX9924+)
- net VR_MAX9924-: now also J30.39 (VR_MAX9924-)
- net WBO_Heater: now also J30.6 (WBO_Heater)
- net WBO_Ip: now also J30.10 (WBO_Ip)
- net WBO_Rtrim: now also J30.13 (WBO_Rtrim)
- net WBO_Un: now also J30.11 (WBO_Un)
- net WBO_Vm: now also J30.12 (WBO_Vm)
Other:
- note added: "SUPERSEAL 1.0 60-pos J30 (TE 6437288-5) replaces the dual AMPSEAL headers and the 2.54 mm 2x02 sockets. Smart-coil only. Pinout: docs/superseal-60-pinout.md."
- note removed: "Dual AMPSEAL 35 redesign: J30 connector A (outputs/power/WBO), J31 connector B (sensors/CAN). Molex Mini-Fit J2 J3 J4 J5 J10 are DNP. Pinout: docs/ampseal-35-pinout.md. Footprint pad geometry is a hypothesis."
