File: uaefi.kicad_pcb (KiCad board)
At the start: 4 copper layers, 158 x 136 mm, 135 parts, among them J30 6437288-5, J6 Conn_01x06, J7 Conn_01x05_Male, J8 USB_B_Mini, J9 USB_C, M1 Module-power_12and5V-0.3, M2 Module-knock-0.2, M3 Module-vr-discrete-0.5, M4 Module-vr-max9924-0.1, M5 Module-wbo-0.5, M6 Module:mega-mcu100/0.3, M7 Module-can-0.1, P1 Pad, P15 Pad, P16 Pad, P17 Pad, P18 Pad, P2 Pad, P3 Pad, P4 Pad, P5 Pad, P6 Pad, P7 Pad, P8 Pad, U1 TLE9201SG, U10 VNLD5160TR-E, U11 VNLD5160TR-E, U2 TLE9201SG, U3 MPX4/MPXH6400_MAP, U4 MAX31855KASA, U5 JDY-33, U6 VNLD5160TR-E, U7 VNLD5160TR-E, U8 VNLD5160TR-E, U9 VNLD5160TR-E

Commit message: Route every SUPERSEAL 60 pin and widen the high-current copper.
The header moves to (214, 78) and the outline grows to 258 by 182 mm so the power and injector runs can leave the pin field. Series widths are documented from the copper on the board, not from the Superseal catalog rating.

Co-authored-by: Quintin <quintinbannink42@users.noreply.github.com>
Parts:
- moved J30 28.0 mm to (214.0, 78.0)
Routing:
- net /WBO_Heater: track 381.0 -> 1377.7 mm, vias 8 -> 21
- net /OUT_INJ2: track 5.71 -> 925.7 mm, vias 0 -> 9
- net /OUT_LS_HOT1: track 341.0 -> 1214.5 mm, vias 8 -> 17
- net +12V: track 500.8 -> 1298.4 mm, vias 11 -> 30
- net /OUT_DC1-: track 376.1 -> 1131.9 mm, vias 5 -> 14
- net +12V_RAW: track 345.4 -> 1093.3 mm, vias 5 -> 25
- net /OUT_LS2: track 350.5 -> 1080.4 mm, vias 10 -> 18
- net /OUT_INJ6: track 404.6 -> 1130.4 mm, vias 11 -> 18
- net /OUT_LS3: track 330.5 -> 1050.5 mm, vias 8 -> 16
- net /12V_KEY: track 548.0 -> 1258.9 mm, vias 11 -> 30
- net /OUT_DC2-: track 249.8 -> 958.1 mm, vias 4 -> 13
- net /OUT_LS4: track 389.3 -> 1081.0 mm, vias 10 -> 18
- net /OUT_INJ3: track 132.6 -> 788.9 mm, vias 3 -> 11
- net /OUT_INJ5: track 129.3 -> 776.0 mm, vias 5 -> 13
- net /OUT_INJ1: track 390.3 -> 1026.1 mm, vias 10 -> 16
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Other:
- board size 158 x 136 mm -> 258 x 182 mm
