File: uaefi.kicad_pcb (KiCad board)
At the start: 4 copper layers, 258 x 182 mm, 135 parts, among them J30 6437288-5, J6 Conn_01x06, J7 Conn_01x05_Male, J8 USB_B_Mini, J9 USB_C, M1 Module-power_12and5V-0.3, M2 Module-knock-0.2, M3 Module-vr-discrete-0.5, M4 Module-vr-max9924-0.1, M5 Module-wbo-0.5, M6 Module:mega-mcu100/0.3, M7 Module-can-0.1, P1 Pad, P15 Pad, P16 Pad, P17 Pad, P18 Pad, P2 Pad, P3 Pad, P4 Pad, P5 Pad, P6 Pad, P7 Pad, P8 Pad, U1 TLE9201SG, U10 VNLD5160TR-E, U11 VNLD5160TR-E, U2 TLE9201SG, U3 MPX4/MPXH6400_MAP, U4 MAX31855KASA, U5 JDY-33, U6 VNLD5160TR-E, U7 VNLD5160TR-E, U8 VNLD5160TR-E, U9 VNLD5160TR-E

Commit message: Move J30 SuperSeal to left edge and shrink outline (#3)
Place the TE 6437288-5 header at (3.5, 138) rotation 90 so the mating shell hangs off the left edge, and pull Edge.Cuts in to 151.2 x 112.1 mm. The 258 x 182 mm right-edge growth is gone. Cavity numbers are unchanged. Harness necks and DRC are recorded in the SuperSeal docs.

Co-authored-by: Cursor Agent <cursoragent@cursor.com>
Co-authored-by: Quintin <quintinbannink42@users.noreply.github.com>
Parts:
- moved J30 218.9 mm to (3.50, 138.0), turned to 90 degrees
Routing:
- net +12V: track 1298.4 -> 74.7 mm, vias 30 -> 1
- net /OUT_LS_HOT1: track 1214.5 -> 67.6 mm, vias 17 -> 5
- net /OUT_DC1-: track 1131.9 -> 65.3 mm, vias 14 -> 5
- net /OUT_INJ6: track 1130.4 -> 65.9 mm, vias 18 -> 2
- net /WBO_Heater: track 1377.7 -> 317.9 mm, vias 21 -> 3
- net /OUT_LS4: track 1081.0 -> 69.0 mm, vias 18 -> 5
- net /OUT_LS2: track 1080.4 -> 68.9 mm, vias 18 -> 3
- net /OUT_LS3: track 1050.5 -> 63.8 mm, vias 16 -> 3
- net /OUT_LS_HOT2: track 1035.2 -> 81.0 mm, vias 11 -> 5
- net /OUT_INJ1: track 1026.1 -> 79.5 mm, vias 16 -> 5
- net /12V_KEY: track 1258.9 -> 351.4 mm, vias 30 -> 8
- net /OUT_DC2-: track 958.1 -> 104.6 mm, vias 13 -> 4
- net /OUT_INJ2: track 925.7 -> 86.7 mm, vias 9 -> 4
- net +12V_RAW: track 1093.3 -> 255.6 mm, vias 25 -> 3
- net /OUT_INJ3: track 788.9 -> 59.0 mm, vias 11 -> 1
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Other:
- board size 258 x 182 mm -> 151.2 x 112.1 mm
- board text added: "J30 SUPERSEAL 6437288-5 on the left edge. Shell hangs off the outline. Smart-coil only. See docs/superseal-60-pinout.md."
- board text removed: "J30 SUPERSEAL 6437288-5 on the right edge. Shell hangs off the outline. Smart-coil only. See docs/superseal-60-pinout.md."
